Commit message: mujoco first integration, swing controller started working

File: description/quadro.xacro (robot description, xacro)
@@ -691,3 +691,81 @@
     <joint_properties friction="0.5"/>
   </joint>
+  <ros2_control name="MujocoSystem" type="system">
+    <hardware>
+      <plugin>mujoco_ros2_control/MujocoSystemInterface</plugin>
+      <param name="mujoco_model">$(find quadruped_control)/description/robot.xml</param>
+    </hardware>
+    <joint name="fl_m1_s1">
+      <command_interface name="effort"/>
+      <state_interface name="position"/>
+      <state_interface name="velocity"/>
+      <state_interface name="effort"/>
+    </joint>
+    <joint name="fl_m2_s2">
+      <command_interface name="effort"/>
+      <state_interface name="position"/>
+      <state_interface name="velocity"/>
+      <state_interface name="effort"/>
+    </joint>
+    <joint name="fl_l4_l3">
+      <command_interface name="effort"/>
+      <state_interface name="position"/>
+      <state_interface name="velocity"/>
+      <state_interface name="effort"/>
+    </joint>
+    <joint name="fr_m1_s1">
+      <command_interface name="effort"/>
+      <state_interface name="position"/>
+      <state_interface name="velocity"/>
+      <state_interface name="effort"/>
+    </joint>
+    <joint name="fr_m2_s2">
+      <command_interface name="effort"/>
+      <state_interface name="position"/>
+      <state_interface name="velocity"/>
+      <state_interface name="effort"/>
+    </joint>
+    <joint name="fr_l4_l3">
+      <command_interface name="effort"/>
+      <state_interface name="position"/>
+      <state_interface name="velocity"/>
+      <state_interface name="effort"/>
+    </joint>
+    <joint name="bl_m1_s1">
+      <command_interface name="effort"/>
+      <state_interface name="position"/>
+      <state_interface name="velocity"/>
+      <state_interface name="effort"/>
+    </joint>
+    <joint name="bl_m2_s2">
+      <command_interface name="effort"/>
+      <state_interface name="position"/>
+      <state_interface name="velocity"/>
+      <state_interface name="effort"/>
+    </joint>
+    <joint name="bl_l4_l3">
+      <command_interface name="effort"/>
+      <state_interface name="position"/>
+      <state_interface name="velocity"/>
+      <state_interface name="effort"/>
+    </joint>
+    <joint name="br_m1_s1">
+      <command_interface name="effort"/>
+      <state_interface name="position"/>
+      <state_interface name="velocity"/>
+      <state_interface name="effort"/>
+    </joint>
+    <joint name="br_m2_s2">
+      <command_interface name="effort"/>
+      <state_interface name="position"/>
+      <state_interface name="velocity"/>
+      <state_interface name="effort"/>
+    </joint>
+    <joint name="br_l4_l3">
+      <command_interface name="effort"/>
+      <state_interface name="position"/>
+      <state_interface name="velocity"/>
+      <state_interface name="effort"/>
+    </joint>
+  </ros2_control>
 </robot>

Commit message: changed robot orientation (base frame)

File: description/quadro.xacro (robot description, xacro)
@@ -6,22 +6,278 @@
   <link name="back_plate">
     <inertial>
-      <origin xyz="-3.82601e-05 -0.00496654 -0.00528261" rpy="0 0 0"/>
+      <origin xyz="0.0139665 -3.82601e-05 -0.0137826" rpy="0 0 0"/>
       <mass value="2.59053"/>
-      <inertia ixx="0.0255846" ixy="-4.15339e-05" ixz="4e-12" iyy="0.00872593" iyz="-0.000207516" izz="0.0313278"/>
-    </inertial>
-    <!-- Part back_plate_parts -->
-    <visual>
-      <origin xyz="-3.82601e-05 -0.00496654 -0.00528261" rpy="0 -0 0"/>
-      <geometry>
-        <mesh filename="file://$(find quadruped_control)/description/assets/back_plate_visual.stl"/>
-      </geometry>
-      <material name="back_plate_parts_material">
-        <color rgba="0.67735 0.643034 0.48069 1"/>
-      </material>
-    </visual>
-    <collision>
-      <origin xyz="-3.82601e-05 -0.00496654 -0.00528261" rpy="0 -0 0"/>
-      <geometry>
-        <mesh filename="file://$(find quadruped_control)/description/assets/back_plate_collision.stl"/>
+      <inertia ixx="0.00872593" ixy="4.15339e-05" ixz="0.000207516" iyy="0.0255846" iyz="8e-12" izz="0.0313278"/>
+    </inertial>
+    <!-- Part back_stop -->
+    <visual>
+      <origin xyz="0.0544675 -3.82602e-05 -0.0584927" rpy="-0 1.652e-09 1.5708"/>
+      <geometry>
+        <mesh filename="file://$(find quadruped_control)/description/assets/back_stop.stl"/>
+      </geometry>
+      <material name="back_stop_material">
+        <color rgba="1 0.756863 0.054902 1"/>
+      </material>
+    </visual>
+    <collision>
+      <origin xyz="0.0544675 -3.82602e-05 -0.0584927" rpy="-0 1.652e-09 1.5708"/>
+      <geometry>
+        <mesh filename="file://$(find quadruped_control)/description/assets/back_stop.stl"/>
+      </geometry>
+    </collision>
+    <!-- Part side_pipe -->
+    <visual>
+      <origin xyz="-0.0846325 -0.147986 -0.0584927" rpy="-0 1.652e-09 1.5708"/>
+      <geometry>
+        <mesh filename="file://$(find quadruped_control)/description/assets/side_pipe.stl"/>
+      </geometry>
+      <material name="side_pipe_material">
+        <color rgba="0 0 0 1"/>
+      </material>
+    </visual>
+    <collision>
+      <origin xyz="-0.0846325 -0.147986 -0.0584927" rpy="-0 1.652e-09 1.5708"/>
+      <geometry>
+        <mesh filename="file://$(find quadruped_control)/description/assets/side_pipe.stl"/>
+      </geometry>
+    </collision>
+    <!-- Part side_cover -->
+    <visual>
+      <origin xyz="0.102368 -3.82602e-05 -0.0584927" rpy="0 -1.652e-09 -1.5708"/>
+      <geometry>
+        <mesh filename="file://$(find quadruped_control)/description/assets/side_cover.stl"/>
+      </geometry>
+      <material name="side_cover_material">
+        <color rgba="0.647059 0.647059 0.647059 1"/>
+      </material>
+    </visual>
+    <collision>
+      <origin xyz="0.102368 -3.82602e-05 -0.0584927" rpy="0 -1.652e-09 -1.5708"/>
+      <geometry>
+        <mesh filename="file://$(find quadruped_control)/description/assets/side_cover.stl"/>
+      </geometry>
+    </collision>
+    <!-- Part back_plate -->
+    <visual>
+      <origin xyz="-0.0846325 -3.82602e-05 -0.0584927" rpy="-0 1.652e-09 1.5708"/>
+      <geometry>
+        <mesh filename="file://$(find quadruped_control)/description/assets/back_plate.stl"/>
+      </geometry>
+      <material name="back_plate_material">
+        <color rgba="1 0.756863 0.054902 1"/>
+      </material>
+    </visual>
+    <collision>
+      <origin xyz="-0.0846325 -3.82602e-05 -0.0584927" rpy="-0 1.652e-09 1.5708"/>
+      <geometry>
+        <mesh filename="file://$(find quadruped_control)/description/assets/back_plate.stl"/>
+      </geometry>
+    </collision>
+    <!-- Part battery -->
+    <visual>
+      <origin xyz="0.0528675 0.0664617 -0.0294927" rpy="1.652e-09 0 -3.14159"/>
+      <geometry>
+        <mesh filename="file://$(find quadruped_control)/description/assets/battery.stl"/>
+      </geometry>
+      <material name="battery_material">
+        <color rgba="0.768627 0.886275 0.952941 1"/>
+      </material>
+    </visual>
+    <collision>
+      <origin xyz="0.0528675 0.0664617 -0.0294927" rpy="1.652e-09 0 -3.14159"/>
+      <geometry>
+        <mesh filename="file://$(find quadruped_control)/description/assets/battery.stl"/>
+      </geometry>
+    </collision>
+    <!-- Part motor -->
+    <visual>
+      <origin xyz="0.113368 -0.0550383 -0.00849266" rpy="3.14159 -0 0"/>
+      <geometry>
+        <mesh filename="file://$(find quadruped_control)/description/assets/motor.stl"/>
+      </geometry>
+      <material name="motor_material">
+        <color rgba="0.498039 0.498039 0.498039 1"/>
+      </material>
+    </visual>
+    <collision>
+      <origin xyz="0.113368 -0.0550383 -0.00849266" rpy="3.14159 -0 0"/>
+      <geometry>
+        <mesh filename="file://$(find quadruped_control)/description/assets/motor.stl"/>
+      </geometry>
+    </collision>
+    <!-- Part side_cover_2 -->
+    <visual>
+      <origin xyz="-0.0846325 -3.82602e-05 -0.0584927" rpy="-0 1.652e-09 1.5708"/>
+      <geometry>
+        <mesh filename="file://$(find quadruped_control)/description/assets/side_cover.stl"/>
+      </geometry>
+      <material name="side_cover_2_material">
+        <color rgba="0.647059 0.647059 0.647059 1"/>
+      </material>
+    </visual>
+    <collision>
+      <origin xyz="-0.0846325 -3.82602e-05 -0.0584927" rpy="-0 1.652e-09 1.5708"/>
+      <geometry>
+        <mesh filename="file://$(find quadruped_control)/description/assets/side_cover.stl"/>
+      </geometry>
+    </collision>
+    <!-- Part motor_2 -->
+    <visual>
+      <origin xyz="-0.0956325 -0.0550383 -0.00849266" rpy="-3.14159 0 -3.14159"/>
+      <geometry>
+        <mesh filename="file://$(find quadruped_control)/description/assets/motor.stl"/>
+      </geometry>
+      <material name="motor_2_material">
+        <color rgba="0.498039 0.498039 0.498039 1"/>
+      </material>
+    </visual>
+    <collision>
+      <origin xyz="-0.0956325 -0.0550383 -0.00849266" rpy="-3.14159 0 -3.14159"/>
+      <geometry>
+        <mesh filename="file://$(find quadruped_control)/description/assets/motor.stl"/>
+      </geometry>
+    </collision>
+    <!-- Part motor_3 -->
+    <visual>
+      <origin xyz="0.113368 0.0549617 -0.00849266" rpy="3.14159 -0 0"/>
+      <geometry>
+        <mesh filename="file://$(find quadruped_control)/description/assets/motor.stl"/>
+      </geometry>
+      <material name="motor_3_material">
+        <color rgba="0.498039 0.498039 0.498039 1"/>
+      </material>
+    </visual>
+    <collision>
+      <origin xyz="0.113368 0.0549617 -0.00849266" rpy="3.14159 -0 0"/>
+      <geometry>
+        <mesh filename="file://$(find quadruped_control)/description/assets/motor.stl"/>
+      </geometry>
+    </collision>
+    <!-- Part bot_pipe_half -->
+    <visual>
+      <origin xyz="-0.418632 -3.82602e-05 -0.0584927" rpy="3.14159 1.652e-09 1.5708"/>
+      <geometry>
+        <mesh filename="file://$(find quadruped_control)/description/assets/bot_pipe_half.stl"/>
+      </geometry>
+      <material name="bot_pipe_half_material">
+        <color rgba="0.972549 0.529412 0.00392157 1"/>
+      </material>
+    </visual>
+    <collision>
+      <origin xyz="-0.418632 -3.82602e-05 -0.0584927" rpy="3.14159 1.652e-09 1.5708"/>
+      <geometry>
+        <mesh filename="file://$(find quadruped_control)/description/assets/bot_pipe_half.stl"/>
+      </geometry>
+    </collision>
+    <!-- Part side_pipe_2 -->
+    <visual>
+      <origin xyz="0.102368 -3.826e-05 0.0955073" rpy="3.14159 1.652e-09 1.5708"/>
+      <geometry>
+        <mesh filename="file://$(find quadruped_control)/description/assets/side_pipe.stl"/>
+      </geometry>
+      <material name="side_pipe_2_material">
+        <color rgba="0 0 0 1"/>
+      </material>
+    </visual>
+    <collision>
+      <origin xyz="0.102368 -3.826e-05 0.0955073" rpy="3.14159 1.652e-09 1.5708"/>
+      <geometry>
+        <mesh filename="file://$(find quadruped_control)/description/assets/side_pipe.stl"/>
+      </geometry>
+    </collision>
+    <!-- Part motor_4 -->
+    <visual>
+      <origin xyz="-0.0956325 0.0549617 -0.00849266" rpy="-3.14159 0 -3.14159"/>
+      <geometry>
+        <mesh filename="file://$(find quadruped_control)/description/assets/motor.stl"/>
+      </geometry>
+      <material name="motor_4_material">
+        <color rgba="0.498039 0.498039 0.498039 1"/>
+      </material>
+    </visual>
+    <collision>
+      <origin xyz="-0.0956325 0.0549617 -0.00849266" rpy="-3.14159 0 -3.14159"/>
+      <geometry>
+        <mesh filename="file://$(find quadruped_control)/description/assets/motor.stl"/>
+      </geometry>
+    </collision>
+    <!-- Part back_stop_2 -->
+    <visual>
+      <origin xyz="-0.0367325 -3.82602e-05 -0.0584927" rpy="0 -1.652e-09 -1.5708"/>
+      <geometry>
+        <mesh filename="file://$(find quadruped_control)/description/assets/back_stop.stl"/>
+      </geometry>
+      <material name="back_stop_2_material">
+        <color rgba="1 0.756863 0.054902 1"/>
+      </material>
+    </visual>
+    <collision>
+      <origin xyz="-0.0367325 -3.82602e-05 -0.0584927" rpy="0 -1.652e-09 -1.5708"/>
+      <geometry>
+        <mesh filename="file://$(find quadruped_control)/description/assets/back_stop.stl"/>
+      </geometry>
+    </collision>
+    <!-- Part back_plate_2 -->
+    <visual>
+      <origin xyz="0.102368 -3.82602e-05 -0.0584927" rpy="0 -1.652e-09 -1.5708"/>
+      <geometry>
+        <mesh filename="file://$(find quadruped_control)/description/assets/back_plate.stl"/>
+      </geometry>
+      <material name="back_plate_2_material">
+        <color rgba="1 0.756863 0.054902 1"/>
+      </material>
+    </visual>
+    <collision>
+      <origin xyz="0.102368 -3.82602e-05 -0.0584927" rpy="0 -1.652e-09 -1.5708"/>
+      <geometry>
+        <mesh filename="file://$(find quadruped_control)/description/assets/back_plate.stl"/>
+      </geometry>
+    </collision>
+    <!-- Part bot_pipe_half_2 -->
+    <visual>
+      <origin xyz="0.436368 -3.82602e-05 -0.0584927" rpy="-0 1.652e-09 1.5708"/>
+      <geometry>
+        <mesh filename="file://$(find quadruped_control)/description/assets/bot_pipe_half.stl"/>
+      </geometry>
+      <material name="bot_pipe_half_2_material">
+        <color rgba="0.972549 0.529412 0.00392157 1"/>
+      </material>
+    </visual>
+    <collision>
+      <origin xyz="0.436368 -3.82602e-05 -0.0584927" rpy="-0 1.652e-09 1.5708"/>
+      <geometry>
+        <mesh filename="file://$(find quadruped_control)/description/assets/bot_pipe_half.stl"/>
+      </geometry>
+    </collision>
+    <!-- Part mid_clamp -->
+    <visual>
+      <origin xyz="-0.224232 -3.82602e-05 -0.0584927" rpy="-0 1.652e-09 1.5708"/>
+      <geometry>
+        <mesh filename="file://$(find quadruped_control)/description/assets/mid_clamp.stl"/>
+      </geometry>
+      <material name="mid_clamp_material">
+        <color rgba="1 0.756863 0.054902 1"/>
+      </material>
+    </visual>
+    <collision>
+      <origin xyz="-0.224232 -3.82602e-05 -0.0584927" rpy="-0 1.652e-09 1.5708"/>
+      <geometry>
+        <mesh filename="file://$(find quadruped_control)/description/assets/mid_clamp.stl"/>
+      </geometry>
+    </collision>
+    <!-- Part battery_2 -->
+    <visual>
+      <origin xyz="0.0528675 -0.0665383 -0.0294927" rpy="-3.14159 0 -3.14159"/>
+      <geometry>
+        <mesh filename="file://$(find quadruped_control)/description/assets/battery.stl"/>
+      </geometry>
+      <material name="battery_2_material">
+        <color rgba="0.768627 0.886275 0.952941 1"/>
+      </material>
+    </visual>
+    <collision>
+      <origin xyz="0.0528675 -0.0665383 -0.0294927" rpy="-3.14159 0 -3.14159"/>
+      <geometry>
+        <mesh filename="file://$(find quadruped_control)/description/assets/battery.stl"/>
       </geometry>
     </collision>
@@ -34,18 +290,50 @@
       <inertia ixx="0.000550761" ixy="-6.00381e-05" ixz="-1.13918e-05" iyy="0.00055728" iyz="1.18589e-05" izz="0.000239291"/>
     </inertial>
-    <!-- Part shaft_parts -->
-    <visual>
-      <origin xyz="-0.00474046 0.00407901 -0.0612986" rpy="-1.5708 0 -3.14159"/>
-      <geometry>
-        <mesh filename="file://$(find quadruped_control)/description/assets/shaft_visual.stl"/>
-      </geometry>
-      <material name="shaft_parts_material">
-        <color rgba="0.556109 0.556109 0.556109 1"/>
-      </material>
-    </visual>
-    <collision>
-      <origin xyz="-0.00474046 0.00407901 -0.0612986" rpy="-1.5708 0 -3.14159"/>
-      <geometry>
-        <mesh filename="file://$(find quadruped_control)/description/assets/shaft_collision.stl"/>
+    <!-- Part lin_1_support_br -->
+    <visual>
+      <origin xyz="-0.019799 0.019799 -0.0735" rpy="0.785398 -1.5708 0"/>
+      <geometry>
+        <mesh filename="file://$(find quadruped_control)/description/assets/lin_1_support_br.stl"/>
+      </geometry>
+      <material name="lin_1_support_br_material">
+        <color rgba="0.901961 0.901961 0.901961 1"/>
+      </material>
+    </visual>
+    <collision>
+      <origin xyz="-0.019799 0.019799 -0.0735" rpy="0.785398 -1.5708 0"/>
+      <geometry>
+        <mesh filename="file://$(find quadruped_control)/description/assets/lin_1_support_br.stl"/>
+      </geometry>
+    </collision>
+    <!-- Part motor_5 -->
+    <visual>
+      <origin xyz="-0.0120208 0.0120208 -0.0735" rpy="-1.5708 0 -0.785398"/>
+      <geometry>
+        <mesh filename="file://$(find quadruped_control)/description/assets/motor.stl"/>
+      </geometry>
+      <material name="motor_5_material">
+        <color rgba="0.498039 0.498039 0.498039 1"/>
+      </material>
+    </visual>
+    <collision>
+      <origin xyz="-0.0120208 0.0120208 -0.0735" rpy="-1.5708 0 -0.785398"/>
+      <geometry>
+        <mesh filename="file://$(find quadruped_control)/description/assets/motor.stl"/>
+      </geometry>
+    </collision>
+    <!-- Part shaft -->
+    <visual>
+      <origin xyz="-0 0 0.01" rpy="1.5708 1.5708 0"/>
+      <geometry>
+        <mesh filename="file://$(find quadruped_control)/description/assets/shaft.stl"/>
+      </geometry>
+      <material name="shaft_material">
+        <color rgba="0.498039 0.498039 0.498039 1"/>
+      </material>
+    </visual>
+    <collision>
+      <origin xyz="-0 0 0.01" rpy="1.5708 1.5708 0"/>
+      <geometry>
+        <mesh filename="file://$(find quadruped_control)/description/assets/shaft.stl"/>
       </geometry>
     </collision>
@@ -58,18 +346,82 @@
       <inertia ixx="0.000439148" ixy="6.14395e-05" ixz="0.000140002" iyy="0.000912333" iyz="-3.78102e-05" izz="0.000883052"/>
     </inertial>
-    <!-- Part shaft_2_parts -->
-    <visual>
-      <origin xyz="0.00931177 -0.00187407 -0.0491985" rpy="-3.14159 -0.785398 1.5708"/>
-      <geometry>
-        <mesh filename="file://$(find quadruped_control)/description/assets/shaft_2_visual.stl"/>
-      </geometry>
-      <material name="shaft_2_parts_material">
-        <color rgba="0.603491 0.603491 0.603491 1"/>
-      </material>
-    </visual>
-    <collision>
-      <origin xyz="0.00931177 -0.00187407 -0.0491985" rpy="-3.14159 -0.785398 1.5708"/>
-      <geometry>
-        <mesh filename="file://$(find quadruped_control)/description/assets/shaft_2_collision.stl"/>
+    <!-- Part bot_r -->
+    <visual>
+      <origin xyz="0 -0 0.1275" rpy="-1.5708 -0 -0.0872665"/>
+      <geometry>
+        <mesh filename="file://$(find quadruped_control)/description/assets/bot_r.stl"/>
+      </geometry>
+      <material name="bot_r_material">
+        <color rgba="0.901961 0.901961 0.901961 1"/>
+      </material>
+    </visual>
+    <collision>
+      <origin xyz="0 -0 0.1275" rpy="-1.5708 -0 -0.0872665"/>
+      <geometry>
+        <mesh filename="file://$(find quadruped_control)/description/assets/bot_r.stl"/>
+      </geometry>
+    </collision>
+    <!-- Part top_r -->
+    <visual>
+      <origin xyz="0 -0 0.1275" rpy="-1.5708 -0 -0.0872665"/>
+      <geometry>
+        <mesh filename="file://$(find quadruped_control)/description/assets/top_r.stl"/>
+      </geometry>
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